Commit message: added joint 4 and 5

File: urdf/devotics_arm.urdf (robot description, URDF)
Before this commit: robot devotics_arm, 4 links, 3 joints
Links:
- added link wrist1_link; visual cylinder length=0.10 radius=0.04
- added link wrist2_link; visual cylinder length=0.10 radius=0.035
Joints:
- added joint joint4: type revolute, parent forearm_link, child wrist1_link, origin xyz=0 0 0.25 rpy=0 0 0, axis 0 1 0, limit lower=-1.57 upper=1.57 effort=10 velocity=1.0
- added joint joint5: type revolute, parent wrist1_link, child wrist2_link, origin xyz=0 0 0.10 rpy=0 0 0, axis 0 0 1, limit lower=-3.14 upper=3.14 effort=10 velocity=1.5

Commit message: added wrist3_link/tool flange is now added and build

File: urdf/devotics_arm.urdf (robot description, URDF)
Before this commit: robot devotics_arm, 6 links, 5 joints
Links:
- added link wrist3_link; visual cylinder length=0.06 radius=0.03
Joints:
- added joint joint6: type revolute, parent wrist2_link, child wrist3_link, origin xyz=0 0 0.10 rpy=0 0 0, axis 0 1 0, limit lower=-3.14 upper=3.14 effort=5 velocity=2.0

Commit message: feat: added left and right figher joint

File: urdf/devotics_arm.urdf (robot description, URDF)
Before this commit: robot devotics_arm, 7 links, 6 joints
Links:
- added link gripper_base_link; visual box size=0.08 0.04 0.04
- added link left_finger_link; visual box size=0.02 0.02 0.06
- added link right_finger_link; visual box size=0.02 0.02 0.06
Joints:
- added joint gripper_base_joint: type fixed, parent wrist3_link, child gripper_base_link, origin xyz=0 0 0.06 rpy=0 0 0
- added joint left_finger_joint: type prismatic, parent gripper_base_link, child left_finger_link, origin xyz=0 0.02 0.04 rpy=0 0 0, axis 0 1 0, limit lower=0.0 upper=0.03 effort=10 velocity=0.1
- added joint right_finger_joint: type prismatic, parent gripper_base_link, child right_finger_link, origin xyz=0 -0.02 0.04 rpy=0 0 0, axis 0 -1 0, limit lower=0.0 upper=0.03 effort=10 velocity=0.1
