Commit message: feat: add IK demonstration script, link collision geometries, and tool0 frame to arm URDF

File: urdf/devotics_arm.urdf.xacro (robot description, xacro)
@@ -81,4 +81,10 @@
             <material name="base_color"/>
         </visual>
+        <collision>
+            <origin xyz="0 0 ${base_length / 2}" rpy="0 0 0"/>
+            <geometry>
+                <cylinder radius="${base_radius}" length="${base_length}"/>
+            </geometry>
+        </collision>
     </link>
     <!-- ============================================================ -->
@@ -93,4 +99,10 @@
             <material name="shoulder_color"/>
         </visual>
+        <collision>
+            <origin xyz="0 0 ${shoulder_size_z / 2}" rpy="0 0 0"/>
+            <geometry>
+                <box size="${shoulder_size_x} ${shoulder_size_y} ${shoulder_size_z}"/>
+            </geometry>
+        </collision>
     </link>
     <joint name="joint1" type="revolute">
@@ -112,4 +124,10 @@
             <material name="upper_arm_color"/>
         </visual>
+        <collision>
+            <origin xyz="0 0 ${upper_arm_length / 2}" rpy="0 0 0"/>
+            <geometry>
+                <box size="${upper_arm_size_x} ${upper_arm_size_y} ${upper_arm_length}"/>
+            </geometry>
+        </collision>
     </link>
     <joint name="joint2" type="revolute">
@@ -131,4 +149,10 @@
             <material name="forearm_color"/>
         </visual>
+        <collision>
+            <origin xyz="0 0 ${forearm_length / 2}" rpy="0 0 0"/>
+            <geometry>
+                <box size="${forearm_size_x} ${forearm_size_y} ${forearm_length}"/>
+            </geometry>
+        </collision>
     </link>
     <joint name="joint3" type="revolute">
@@ -150,4 +174,10 @@
             <material name="wrist1_color"/>
         </visual>
+        <collision>
+            <origin xyz="0 0 ${wrist1_length / 2}" rpy="0 0 0"/>
+            <geometry>
+                <cylinder radius="${wrist1_radius}" length="${wrist1_length}"/>
+            </geometry>
+        </collision>
     </link>
     <joint name="joint4" type="revolute">
@@ -169,4 +199,10 @@
             <material name="wrist2_color"/>
         </visual>
+        <collision>
+            <origin xyz="0 0 ${wrist2_length / 2}" rpy="0 0 0"/>
+            <geometry>
+                <cylinder radius="${wrist2_radius}" length="${wrist2_length}"/>
+            </geometry>
+        </collision>
     </link>
     <joint name="joint5" type="revolute">
@@ -188,4 +224,10 @@
             <material name="wrist3_color"/>
         </visual>
+        <collision>
+            <origin xyz="0 0 ${wrist3_length / 2}" rpy="0 0 0"/>
+            <geometry>
+                <cylinder radius="${wrist3_radius}" length="${wrist3_length}"/>
+            </geometry>
+        </collision>
     </link>
     <joint name="joint6" type="revolute">
@@ -207,4 +249,10 @@
             <material name="gripper_base_color"/>
         </visual>
+        <collision>
+            <origin xyz="0 0 0.02" rpy="0 0 0"/>
+            <geometry>
+                <box size="0.08 0.04 0.04"/>
+            </geometry>
+        </collision>
     </link>
     <joint name="gripper_base_joint" type="fixed">
@@ -224,4 +272,10 @@
             <material name="finger_color"/>
         </visual>
+        <collision>
+            <origin xyz="0 0 ${finger_size_z / 2}" rpy="0 0 0"/>
+            <geometry>
+                <box size="${finger_size_x} ${finger_size_y} ${finger_size_z}"/>
+            </geometry>
+        </collision>
     </link>
     <joint name="left_finger_joint" type="prismatic">
@@ -240,4 +294,10 @@
             <material name="finger_color"/>
         </visual>
+        <collision>
+            <origin xyz="0 0 ${finger_size_z / 2}" rpy="0 0 0"/>
+            <geometry>
+                <box size="${finger_size_x} ${finger_size_y} ${finger_size_z}"/>
+            </geometry>
+        </collision>
     </link>
     <joint name="right_finger_joint" type="prismatic">
@@ -248,3 +308,13 @@
         <limit lower="0.0" upper="${finger_stroke}" effort="10" velocity="0.1"/>
     </joint>
+    <!-- ============================================================ -->
+    <!-- TOOL CENTER POINT (TCP / tool0)                              -->
+    <!-- Virtual frame at the grasp center between finger tips        -->
+    <!-- ============================================================ -->
+    <link name="tool0"/>
+    <joint name="tool0_joint" type="fixed">
+        <parent link="gripper_base_link"/>
+        <child link="tool0"/>
+        <origin xyz="0 0 0.10" rpy="0 0 0"/>
+    </joint>
 </robot>
