Commit message: Phase 3 (Days 21-25): Added gripper hardware interface, multi-controller management, and autonomous pick_and_place.py

File: urdf/devotics_arm.ros2_control.xacro (robot description, xacro)
@@ -48,4 +48,20 @@
         <state_interface name="velocity"/>
       </joint>
+       <!-- LEFT FINGER -->
+      <joint name="left_finger_joint">
+        <command_interface name="position"/>
+        <state_interface name="position">
+          <param name="initial_value">0.0</param>
+        </state_interface>
+        <state_interface name="velocity"/>
+      </joint>
+      <!-- RIGHT FINGER -->
+      <joint name="right_finger_joint">
+        <command_interface name="position"/>
+        <state_interface name="position">
+          <param name="initial_value">0.0</param>
+        </state_interface>
+        <state_interface name="velocity"/>
+      </joint>
     </ros2_control>
   </xacro:macro>

Commit message: Phase 4 (Days 26-30): Gazebo Harmonic physics simulation, mass & inertia, world anchor, and table_cube SDF world

File: urdf/devotics_arm.ros2_control.xacro (robot description, xacro)
@@ -1,8 +1,13 @@
 <?xml version="1.0"?>
 <robot xmlns:xacro="http://www.ros.org/wiki/xacro">
-  <xacro:macro name="devotics_arm_ros2_control" params="name">
+  <xacro:macro name="devotics_arm_ros2_control" params="name sim_mode:=false">
     <ros2_control name="${name}" type="system">
       <hardware>
-        <plugin>mock_components/GenericSystem</plugin>
+        <xacro:if value="${sim_mode}">
+          <plugin>gz_ros2_control/GazeboSimSystem</plugin>
+        </xacro:if>
+        <xacro:unless value="${sim_mode}">
+          <plugin>mock_components/GenericSystem</plugin>
+        </xacro:unless>
       </hardware>
       <joint name="joint1">
@@ -48,5 +53,5 @@
         <state_interface name="velocity"/>
       </joint>
-       <!-- LEFT FINGER -->
+      <!-- LEFT FINGER -->
       <joint name="left_finger_joint">
         <command_interface name="position"/>

File: urdf/devotics_arm.urdf.xacro (robot description, xacro)
@@ -1,4 +1,5 @@
 <?xml version="1.0"?>
 <robot name="devotics_arm" xmlns:xacro="http://www.ros.org/wiki/xacro">
+<xacro:arg name="sim_mode" default="false"/>
     <!-- ============================================================ -->
     <!-- CONSTANTS & PROPERTIES                                       -->
@@ -40,4 +41,27 @@
     <xacro:property name="j6_lower" value="-3.14"/>
     <xacro:property name="j6_upper" value="3.14"/>
+        <!-- INERTIA MACROS -->
+    <xacro:macro name="cylinder_inertia" params="mass radius length *origin">
+        <inertial>
+            <xacro:insert_block name="origin"/>
+            <mass value="${mass}"/>
+            <inertia
+                ixx="${mass*(3*radius*radius + length*length)/12}"
+                iyy="${mass*(3*radius*radius + length*length)/12}"
+                izz="${mass*radius*radius/2}"
+                ixy="0" ixz="0" iyz="0"/>
+        </inertial>
+    </xacro:macro>
+    <xacro:macro name="box_inertia" params="mass x y z *origin">
+        <inertial>
+            <xacro:insert_block name="origin"/>
+            <mass value="${mass}"/>
+            <inertia
+                ixx="${mass*(y*y + z*z)/12}"
+                iyy="${mass*(x*x + z*z)/12}"
+                izz="${mass*(x*x + y*y)/12}"
+                ixy="0" ixz="0" iyz="0"/>
+        </inertial>
+    </xacro:macro>
     <!-- ============================================================ -->
     <!-- MATERIALS                                                    -->
@@ -87,5 +111,15 @@
             </geometry>
         </collision>
-    </link>
+        <xacro:cylinder_inertia mass="2.5" radius="${base_radius}" length="${base_length}">
+            <origin xyz="0 0 ${base_length/2}" rpy="0 0 0"/>
+        </xacro:cylinder_inertia>
+    </link>
+        <!-- WORLD LINK (Anchors the robot base to the Gazebo ground) -->
+    <link name="world"/>
+    <joint name="world_to_base_joint" type="fixed">
+        <parent link="world"/>
+        <child link="base_link"/>
+        <origin xyz="0 0 0" rpy="0 0 0"/>
+    </joint>
     <!-- ============================================================ -->
     <!-- SHOULDER LINK & JOINT 1                                      -->
@@ -105,4 +139,7 @@
             </geometry>
         </collision>
+        <xacro:box_inertia mass="1.2" x="0.12" y="0.12" z="0.10">
+            <origin xyz="0 0 0.05" rpy="0 0 0"/>
+        </xacro:box_inertia>
     </link>
     <joint name="joint1" type="revolute">
@@ -130,4 +167,7 @@
             </geometry>
         </collision>
+        <xacro:box_inertia mass="0.9" x="${upper_arm_size_x}" y="${upper_arm_size_y}" z="${upper_arm_length}">
+            <origin xyz="0 0 ${upper_arm_length/2}" rpy="0 0 0"/>
+        </xacro:box_inertia>
     </link>
     <joint name="joint2" type="revolute">
@@ -155,4 +195,7 @@
             </geometry>
         </collision>
+        <xacro:box_inertia mass="0.7" x="${forearm_size_x}" y="${forearm_size_y}" z="${forearm_length}">
+            <origin xyz="0 0 ${forearm_length/2}" rpy="0 0 0"/>
+        </xacro:box_inertia>
     </link>
     <joint name="joint3" type="revolute">
@@ -180,4 +223,7 @@
             </geometry>
         </collision>
+        <xacro:cylinder_inertia mass="0.3" radius="0.04" length="0.10">
+            <origin xyz="0 0 0.05" rpy="0 0 0"/>
+        </xacro:cylinder_inertia>
     </link>
     <joint name="joint4" type="revolute">
@@ -205,4 +251,7 @@
             </geometry>
         </collision>
+        <xacro:cylinder_inertia mass="0.25" radius="0.035" length="0.10">
+            <origin xyz="0 0 0.05" rpy="0 0 0"/>
+        </xacro:cylinder_inertia>
     </link>
     <joint name="joint5" type="revolute">
@@ -230,4 +279,7 @@
             </geometry>
         </collision>
+        <xacro:cylinder_inertia mass="0.15" radius="0.03" length="0.06">
+            <origin xyz="0 0 0.03" rpy="0 0 0"/>
+        </xacro:cylinder_inertia>
     </link>
     <joint name="joint6" type="revolute">
@@ -255,4 +307,7 @@
             </geometry>
         </collision>
+        <xacro:box_inertia mass="0.2" x="0.08" y="0.04" z="0.04">
+            <origin xyz="0 0 0.02" rpy="0 0 0"/>
+        </xacro:box_inertia>
     </link>
     <joint name="gripper_base_joint" type="fixed">
@@ -278,4 +333,7 @@
             </geometry>
         </collision>
+        <xacro:box_inertia mass="0.05" x="0.02" y="0.02" z="0.06">
+            <origin xyz="0 0.02 0.03" rpy="0 0 0"/>
+        </xacro:box_inertia>
     </link>
     <joint name="left_finger_joint" type="prismatic">
@@ -300,4 +358,7 @@
             </geometry>
         </collision>
+        <xacro:box_inertia mass="0.05" x="0.02" y="0.02" z="0.06">
+            <origin xyz="0 -0.02 0.03" rpy="0 0 0"/>
+        </xacro:box_inertia>
     </link>
     <joint name="right_finger_joint" type="prismatic">
@@ -321,5 +382,11 @@
     <!-- ROS2_CONTROL HARDWARE INTERFACE (MOCK SYSTEM)                -->
     <!-- ============================================================ -->
-    <xacro:include filename="$(find devotics_arm_description)/urdf/devotics_arm.ros2_control.xacro"/>
-    <xacro:devotics_arm_ros2_control name="DevoticsArmMockHardware"/>
+    <xacro:include filename="devotics_arm.ros2_control.xacro"/>
+<xacro:devotics_arm_ros2_control name="DevoticsMockHardware" sim_mode="$(arg sim_mode)"/>
+<!-- Gazebo ROS 2 Control Plugin -->
+<gazebo>
+    <plugin filename="gz_ros2_control-system" name="gz_ros2_control::GazeboSimROS2ControlPlugin">
+        <parameters>$(find devotics_arm_moveit_config)/config/ros2_controllers.yaml</parameters>
+    </plugin>
+</gazebo>
 </robot>
