Commit message: feat: add MoveIt configuration and analytical IK scripts, and update robot physical dimensions and calibration

File: urdf/devotics_arm_v0.urdf.xacro (robot description, xacro)
@@ -58,28 +58,23 @@
   <!-- ============================================================ -->
   <!--
-    F = table surface → J1 rotation axis  (vertical height, mm)
-    MEASUREMENT PENDING — replace 0.042 with real value
-  -->
-  <xacro:property name="dim_F"  value="0.042"/>  <!-- PLACEHOLDER: measure F -->
-  <!--
-    A = J1 rotation axis → J2 (shoulder) axis  (vertical, in rotating base frame)
-    MEASUREMENT PENDING — replace 0.038 with real value
-  -->
-  <xacro:property name="dim_A"  value="0.038"/>  <!-- PLACEHOLDER: measure A -->
-  <!--
-    B = J2 (shoulder) axis → J3 (elbow) axis  (along upper arm)
-    CAD-derived estimate ≈ 38.9 mm — VERIFY ON PHYSICAL ROBOT
-  -->
-  <xacro:property name="dim_B"  value="0.0389"/>  <!-- CAD ~38.9mm: verify B -->
-  <!--
-    C = J3 (elbow) axis → J4 / gripper reference (along forearm)
-    MEASUREMENT PENDING — replace 0.040 with real value
-  -->
-  <xacro:property name="dim_C"  value="0.040"/>  <!-- PLACEHOLDER: measure C -->
-  <!--
-    D = J4 / gripper axis → fingertip  (gripper effective length)
-    MEASUREMENT PENDING — replace 0.030 with real value
-  -->
-  <xacro:property name="dim_D"  value="0.030"/>  <!-- PLACEHOLDER: measure D -->
+    F = table surface → J1 rotation axis  (vertical height, 3.0 cm)
+  -->
+  <xacro:property name="dim_F"  value="0.030"/>  <!-- Physically verified: 3.0 cm -->
+  <!--
+    A = J1 rotation axis → J2 (shoulder) axis  (vertical, 2.5 cm)
+  -->
+  <xacro:property name="dim_A"  value="0.025"/>  <!-- Physically verified: 2.5 cm -->
+  <!--
+    B = J2 (shoulder) axis → J3 (elbow) axis  (along upper arm, 4.0 cm)
+  -->
+  <xacro:property name="dim_B"  value="0.040"/>  <!-- Physically verified: 4.0 cm -->
+  <!--
+    C = J3 (elbow) axis → J4 / gripper reference (along forearm, 4.0 cm)
+  -->
+  <xacro:property name="dim_C"  value="0.040"/>  <!-- Physically verified: 4.0 cm -->
+  <!--
+    D = J4 / gripper axis → fingertip  (gripper effective length, 4.5 cm)
+  -->
+  <xacro:property name="dim_D"  value="0.045"/>  <!-- Physically verified: 4.5 cm (Total upright height = 18.0 cm) -->
   <!-- ============================================================ -->
   <!-- JOINT LIMITS                                                 -->
@@ -92,10 +87,10 @@
   <xacro:property name="j1_lower"  value="${-60.0 * pi / 180.0}"/>
   <xacro:property name="j1_upper"  value="${ 60.0 * pi / 180.0}"/>
-  <!-- J2 shoulder: servo 60–150°  → ROS -30° to +60° = -0.524 to +1.047 rad -->
+  <!-- J2 shoulder: servo 60–175°  → ROS -30° to +85° = -0.524 to +1.484 rad -->
   <xacro:property name="j2_lower"  value="${-30.0 * pi / 180.0}"/>
-  <xacro:property name="j2_upper"  value="${ 60.0 * pi / 180.0}"/>
-  <!-- J3 elbow:    servo 60–150°  → ROS -30° to +60° = -0.524 to +1.047 rad -->
+  <xacro:property name="j2_upper"  value="${ 85.0 * pi / 180.0}"/>
+  <!-- J3 elbow:    servo 60–175°  → ROS -30° to +85° = -0.524 to +1.484 rad -->
   <xacro:property name="j3_lower"  value="${-30.0 * pi / 180.0}"/>
-  <xacro:property name="j3_upper"  value="${ 60.0 * pi / 180.0}"/>
+  <xacro:property name="j3_upper"  value="${ 85.0 * pi / 180.0}"/>
   <!-- J4 gripper:  servo 60–110°  → ROS -30° to +20° = -0.524 to +0.349 rad -->
   <!-- negative = closes (servo < 90°), positive = opens (servo > 90°)        -->

Commit message: feat: add 3D mesh files and update URDF visual geometries for arm components

File: urdf/devotics_arm_v0.urdf.xacro (robot description, xacro)
@@ -133,7 +133,8 @@
   <link name="base_link">
     <visual>
-      <origin xyz="0 0 ${base_stl_height / 2.0}" rpy="0 0 0"/>
-      <geometry>
-        <box size="${base_width} ${base_depth} ${base_stl_height}"/>
+      <!-- Real 3D Printed Base Bracket -->
+      <origin xyz="0 0 0" rpy="0 0 0"/>
+      <geometry>
+        <mesh filename="package://devotics_arm_description/meshes/v0/base/base_bracket.stl" scale="0.001 0.001 0.001"/>
       </geometry>
       <material name="v0_dark_gray"/>
@@ -173,8 +174,15 @@
   <link name="base_rotating_link">
     <visual>
-      <!-- Visual: column from J1 axis up to J2 axis -->
-      <origin xyz="0 0 ${dim_A / 2.0}" rpy="0 0 0"/>
-      <geometry>
-        <box size="${arm_w} ${arm_d} ${dim_A}"/>
+      <!-- Rotating Tower Housing -->
+      <origin xyz="0 0 0" rpy="0 0 0"/>
+      <geometry>
+        <mesh filename="package://devotics_arm_description/meshes/v0/base/housing_left.stl" scale="0.001 0.001 0.001"/>
+      </geometry>
+      <material name="v0_dark_blue"/>
+    </visual>
+    <visual>
+      <origin xyz="0 0 0" rpy="0 0 0"/>
+      <geometry>
+        <mesh filename="package://devotics_arm_description/meshes/v0/base/housing_right.stl" scale="0.001 0.001 0.001"/>
       </geometry>
       <material name="v0_dark_blue"/>
@@ -213,7 +221,7 @@
   <link name="upper_arm_link">
     <visual>
-      <origin xyz="0 0 ${dim_B / 2.0}" rpy="0 0 0"/>
-      <geometry>
-        <box size="${arm_w} ${arm_d} ${dim_B}"/>
+      <origin xyz="0 0 0" rpy="0 0 0"/>
+      <geometry>
+        <mesh filename="package://devotics_arm_description/meshes/v0/arm/bracket_upper_left.stl" scale="0.001 0.001 0.001"/>
       </geometry>
       <material name="v0_mid_blue"/>
@@ -252,7 +260,7 @@
   <link name="forearm_link">
     <visual>
-      <origin xyz="0 0 ${dim_C / 2.0}" rpy="0 0 0"/>
-      <geometry>
-        <box size="${arm_w} ${arm_d} ${dim_C}"/>
+      <origin xyz="0 0 0" rpy="0 0 0"/>
+      <geometry>
+        <mesh filename="package://devotics_arm_description/meshes/v0/arm/bracket_left.stl" scale="0.001 0.001 0.001"/>
       </geometry>
       <material name="v0_orange"/>
@@ -291,7 +299,7 @@
   <link name="gripper_link">
     <visual>
-      <origin xyz="0 0 ${gripper_size_z / 2.0}" rpy="0 0 0"/>
-      <geometry>
-        <box size="${gripper_size_x} ${gripper_size_y} ${gripper_size_z}"/>
+      <origin xyz="0 0 0" rpy="0 0 0"/>
+      <geometry>
+        <mesh filename="package://devotics_arm_description/meshes/v0/gripper/gripper_housing.stl" scale="0.001 0.001 0.001"/>
       </geometry>
       <material name="v0_light_gray"/>

Commit message: feat: add new arm bracket meshes and update URDF model components

File: urdf/devotics_arm_v0.urdf.xacro (robot description, xacro)
@@ -62,7 +62,7 @@
   <xacro:property name="dim_F"  value="0.030"/>  <!-- Physically verified: 3.0 cm -->
   <!--
-    A = J1 rotation axis → J2 (shoulder) axis  (vertical, 2.5 cm)
-  -->
-  <xacro:property name="dim_A"  value="0.025"/>  <!-- Physically verified: 2.5 cm -->
+    A = J1 rotation axis → J2 (shoulder) axis  (vertical, 6.02 cm to upper housing pivot)
+  -->
+  <xacro:property name="dim_A"  value="0.0602"/>  <!-- Matched to CAD housing upper pivot -->
   <!--
     B = J2 (shoulder) axis → J3 (elbow) axis  (along upper arm, 4.0 cm)
@@ -131,10 +131,13 @@
   <!-- Visual: CAD bounding box (72.24 × 70.58 × 28.59 mm).       -->
   <!-- ============================================================ -->
+    <!-- ============================================================ -->
+  <!-- BASE LINK                                                    -->
+  <!-- Fixed base that sits on the table surface (Z=0).            -->
+  <!-- ============================================================ -->
   <link name="base_link">
     <visual>
-      <!-- Real 3D Printed Base Bracket -->
-      <origin xyz="0 0 0" rpy="0 0 0"/>
-      <geometry>
-        <mesh filename="package://devotics_arm_description/meshes/v0/base/base_bracket.stl" scale="0.001 0.001 0.001"/>
+      <origin xyz="0 0 ${base_stl_height / 2.0}" rpy="0 0 0"/>
+      <geometry>
+        <box size="${base_width} ${base_depth} ${base_stl_height}"/>
       </geometry>
       <material name="v0_dark_gray"/>
@@ -149,17 +152,10 @@
   <!-- ============================================================ -->
   <!-- J1 — BASE ROTATION JOINT                                     -->
-  <!-- Rotates the entire arm around the vertical (Z) axis.         -->
-  <!-- Origin at J1 servo shaft center, height F above table.      -->
-  <!-- dim_F = PENDING measurement                                  -->
   <!-- ============================================================ -->
   <joint name="base_joint" type="revolute">
     <parent link="base_link"/>
     <child  link="base_rotating_link"/>
-    <!--
-      xyz: Z = dim_F (table → J1 axis height) — PENDING MEASUREMENT
-      Once F is measured, update dim_F above.
-    -->
     <origin xyz="0 0 ${dim_F}" rpy="0 0 0"/>
-    <axis xyz="0 0 1"/>  <!-- Z: vertical rotation -->
+    <axis xyz="0 0 1"/>
     <limit lower="${j1_lower}" upper="${j1_upper}" effort="1.5" velocity="1.8"/>
     <dynamics damping="0.01" friction="0.01"/>
@@ -167,13 +163,17 @@
   <!-- ============================================================ -->
   <!-- BASE ROTATING LINK                                           -->
-  <!-- The part of the arm that rotates with J1.                   -->
-  <!-- Its origin is at the J1 axis.                               -->
-  <!-- Extends upward to the J2 (shoulder) axis: height = dim_A.  -->
-  <!-- dim_A = PENDING measurement                                 -->
   <!-- ============================================================ -->
   <link name="base_rotating_link">
-    <visual>
-      <!-- Rotating Tower Housing -->
-      <origin xyz="0 0 0" rpy="0 0 0"/>
+    <!-- Servo horn mounting plate at base (flat on base platform) -->
+    <visual>
+      <origin xyz="0.05828 0 -0.04365" rpy="0 0 -1.5708"/>
+      <geometry>
+        <mesh filename="package://devotics_arm_description/meshes/v0/base/horn_base.stl" scale="0.001 0.001 0.001"/>
+      </geometry>
+      <material name="v0_dark_gray"/>
+    </visual>
+    <!-- Left housing upright (100% vertical along +Z, seated flush on base) -->
+    <visual>
+      <origin xyz="0.08918 0 0.00592" rpy="0.7944 0 -1.5708"/>
       <geometry>
         <mesh filename="package://devotics_arm_description/meshes/v0/base/housing_left.stl" scale="0.001 0.001 0.001"/>
@@ -181,6 +181,7 @@
       <material name="v0_dark_blue"/>
     </visual>
-    <visual>
-      <origin xyz="0 0 0" rpy="0 0 0"/>
+    <!-- Right housing upright (100% vertical along +Z, seated flush on base) -->
+    <visual>
+      <origin xyz="0.08918 0 0.00592" rpy="0.7944 0 -1.5708"/>
       <geometry>
         <mesh filename="package://devotics_arm_description/meshes/v0/base/housing_right.stl" scale="0.001 0.001 0.001"/>
@@ -188,4 +189,36 @@
       <material name="v0_dark_blue"/>
     </visual>
+    <!-- Lower Left Bracket (exact CAD assembly match) -->
+    <visual>
+      <origin xyz="0.08918 0 0.00592" rpy="0.7944 0 -1.5708"/>
+      <geometry>
+        <mesh filename="package://devotics_arm_description/meshes/v0/arm/bracket_lower_left.stl" scale="0.001 0.001 0.001"/>
+      </geometry>
+      <material name="v0_light_gray"/>
+    </visual>
+    <!-- Lower Right Bracket (exact CAD assembly match) -->
+    <visual>
+      <origin xyz="0.08918 0 0.00592" rpy="0.7944 0 -1.5708"/>
+      <geometry>
+        <mesh filename="package://devotics_arm_description/meshes/v0/arm/bracket_lower_right.stl" scale="0.001 0.001 0.001"/>
+      </geometry>
+      <material name="v0_light_gray"/>
+    </visual>
+    <!-- Upper Left Bracket (exact CAD assembly match) -->
+    <visual>
+      <origin xyz="0.08918 0 0.00592" rpy="0.7944 0 -1.5708"/>
+      <geometry>
+        <mesh filename="package://devotics_arm_description/meshes/v0/arm/bracket_upper_left.stl" scale="0.001 0.001 0.001"/>
+      </geometry>
+      <material name="v0_light_gray"/>
+    </visual>
+    <!-- Upper Right Bracket (exact CAD assembly match) -->
+    <visual>
+      <origin xyz="0.08918 0 0.00592" rpy="0.7944 0 -1.5708"/>
+      <geometry>
+        <mesh filename="package://devotics_arm_description/meshes/v0/arm/bracket_upper_right.stl" scale="0.001 0.001 0.001"/>
+      </geometry>
+      <material name="v0_light_gray"/>
+    </visual>
     <collision>
       <origin xyz="0 0 ${dim_A / 2.0}" rpy="0 0 0"/>
@@ -197,17 +230,10 @@
   <!-- ============================================================ -->
   <!-- J2 — SHOULDER JOINT                                          -->
-  <!-- Pitches the upper arm forward/backward.                     -->
-  <!-- Origin at J2 servo shaft center, height A above J1 axis.   -->
-  <!-- dim_A = PENDING measurement                                 -->
-  <!-- Axis: Y  (positive = arm moves forward/down per firmware)   -->
   <!-- ============================================================ -->
   <joint name="shoulder_joint" type="revolute">
     <parent link="base_rotating_link"/>
     <child  link="upper_arm_link"/>
-    <!--
-      xyz: Z = dim_A (J1 axis → J2 axis height) — PENDING MEASUREMENT
-    -->
     <origin xyz="0 0 ${dim_A}" rpy="0 0 0"/>
-    <axis xyz="0 1 0"/>  <!-- Y: pitch axis -->
+    <axis xyz="0 1 0"/>
     <limit lower="${j2_lower}" upper="${j2_upper}" effort="1.5" velocity="1.8"/>
     <dynamics damping="0.01" friction="0.01"/>
@@ -215,13 +241,10 @@
   <!-- ============================================================ -->
   <!-- UPPER ARM LINK                                               -->
-  <!-- Connects shoulder (J2) to elbow (J3).                       -->
-  <!-- Origin at J2 axis. Length = dim_B (~38.9mm from CAD).       -->
-  <!-- dim_B = CAD estimate — verify on physical robot.            -->
   <!-- ============================================================ -->
   <link name="upper_arm_link">
     <visual>
-      <origin xyz="0 0 0" rpy="0 0 0"/>
-      <geometry>
-        <mesh filename="package://devotics_arm_description/meshes/v0/arm/bracket_upper_left.stl" scale="0.001 0.001 0.001"/>
+      <origin xyz="0 0 ${dim_B / 2.0}" rpy="0 0 0"/>
+      <geometry>
+        <box size="${arm_w} ${arm_d} ${dim_B}"/>
       </geometry>
       <material name="v0_mid_blue"/>
@@ -236,17 +259,10 @@
   <!-- ============================================================ -->
   <!-- J3 — ELBOW JOINT                                             -->
-  <!-- Bends the forearm relative to the upper arm.                -->
-  <!-- Origin at J3 servo shaft center, distance B from J2 axis.  -->
-  <!-- Axis: Y  (positive = forearm moves forward/down per firmware)-->
   <!-- ============================================================ -->
   <joint name="elbow_joint" type="revolute">
     <parent link="upper_arm_link"/>
     <child  link="forearm_link"/>
-    <!--
-      xyz: Z = dim_B (J2 axis → J3 axis distance along upper arm)
-      dim_B ≈ 38.9mm from CAD — verify on robot.
-    -->
     <origin xyz="0 0 ${dim_B}" rpy="0 0 0"/>
-    <axis xyz="0 1 0"/>  <!-- Y: pitch axis -->
+    <axis xyz="0 1 0"/>
     <limit lower="${j3_lower}" upper="${j3_upper}" effort="1.5" velocity="1.8"/>
     <dynamics damping="0.01" friction="0.01"/>
@@ -254,13 +270,10 @@
   <!-- ============================================================ -->
   <!-- FOREARM LINK                                                 -->
-  <!-- Connects elbow (J3) to gripper (J4) reference.             -->
-  <!-- Origin at J3 axis. Length = dim_C.                          -->
-  <!-- dim_C = PENDING measurement                                 -->
   <!-- ============================================================ -->
   <link name="forearm_link">
     <visual>
-      <origin xyz="0 0 0" rpy="0 0 0"/>
-      <geometry>
-        <mesh filename="package://devotics_arm_description/meshes/v0/arm/bracket_left.stl" scale="0.001 0.001 0.001"/>
+      <origin xyz="0 0 ${dim_C / 2.0}" rpy="0 0 0"/>
+      <geometry>
+        <box size="${arm_w} ${arm_d} ${dim_C}"/>
       </geometry>
       <material name="v0_orange"/>
@@ -275,18 +288,10 @@
   <!-- ============================================================ -->
   <!-- J4 — GRIPPER JOINT                                           -->
-  <!-- Opens and closes the gripper via the J4 MG90S servo.        -->
-  <!-- This is NOT a positioning DOF — it is the gripper actuator. -->
-  <!-- Origin at J4 servo shaft center, distance C from J3 axis.  -->
-  <!-- dim_C = PENDING measurement                                 -->
   <!-- ============================================================ -->
   <joint name="gripper_joint" type="revolute">
     <parent link="forearm_link"/>
     <child  link="gripper_link"/>
-    <!--
-      xyz: Z = dim_C (J3 axis → J4/gripper reference) — PENDING MEASUREMENT
-    -->
     <origin xyz="0 0 ${dim_C}" rpy="0 0 0"/>
     <axis xyz="0 1 0"/>
-    <!-- negative = closes, positive = opens -->
     <limit lower="${j4_lower}" upper="${j4_upper}" effort="0.5" velocity="1.5"/>
     <dynamics damping="0.005" friction="0.005"/>
@@ -294,27 +299,22 @@
   <!-- ============================================================ -->
   <!-- GRIPPER LINK                                                 -->
-  <!-- The gripper servo housing. Bounding box from CAD/STL.       -->
-  <!-- 19.60 × 37.35 × 27.63 mm                                   -->
   <!-- ============================================================ -->
   <link name="gripper_link">
     <visual>
-      <origin xyz="0 0 0" rpy="0 0 0"/>
-      <geometry>
-        <mesh filename="package://devotics_arm_description/meshes/v0/gripper/gripper_housing.stl" scale="0.001 0.001 0.001"/>
-      </geometry>
-      <material name="v0_light_gray"/>
-    </visual>
-    <collision>
       <origin xyz="0 0 ${gripper_size_z / 2.0}" rpy="0 0 0"/>
       <geometry>
         <box size="${gripper_size_x} ${gripper_size_y} ${gripper_size_z}"/>
       </geometry>
+      <material name="v0_light_gray"/>
+    </visual>
+    <collision>
+      <origin xyz="0 0 ${gripper_size_z / 2.0}" rpy="0 0 0"/>
+      <geometry>
+        <box size="${gripper_size_x} ${gripper_size_y} ${gripper_size_z}"/>
+      </geometry>
     </collision>
   </link>
   <!-- ============================================================ -->
   <!-- TOOL CENTER POINT (tool0)                                    -->
-  <!-- Virtual frame at the fingertip / grasp center.              -->
-  <!-- This is the end-effector reference for forward/inverse IK.  -->
-  <!-- dim_D = PENDING measurement                                 -->
   <!-- ============================================================ -->
   <link name="tool0"/>
@@ -322,7 +322,4 @@
     <parent link="gripper_link"/>
     <child  link="tool0"/>
-    <!--
-      xyz: Z = dim_D (J4/gripper axis → fingertip) — PENDING MEASUREMENT
-    -->
     <origin xyz="0 0 ${dim_D}" rpy="0 0 0"/>
   </joint>
